Commit message: new file:   .vendored-hashes.txt new file:   LICENSE new file:   README new file:   README.md new file:   champ/.gitmodules new file:   champ/.travis.yml new file:   champ/LICENSE new file:   champ/README.md new file:   champ/champ/CMakeLists.txt new file:   champ/champ/include/champ/LICENSE new file:   champ/champ/include/champ/README.md new file:   champ/champ/include/champ/bla/basic_linear_algebra.h new file:   champ/champ/include/champ/bla/memory_delegate.h new file:   champ/champ/include/champ/body_controller/body_controller.h new file:   champ/champ/include/champ/geometry/geometry.h new file:   champ/champ/include/champ/kinematics/kinematics.h new file:   champ/champ/include/champ/leg_controller/leg_controller.h new file:   champ/champ/include/champ/leg_controller/phase_generator.h new file:   champ/champ/include/champ/leg_controller/trajectory_planner.h new file:   champ/champ/include/champ/macros/macros.h new file:   champ/champ/include/champ/odometry/odometry.h new file:   champ/champ/include/champ/quadruped_base/quadruped_base.h new file:   champ/champ/include/champ/quadruped_base/quadruped_components.h new file:   champ/champ/include/champ/quadruped_base/quadruped_joint.h new file:   champ/champ/include/champ/quadruped_base/quadruped_leg.h new file:   champ/champ/include/champ/utils/urdf_loader.h new file:   champ/champ/include/champ/utils/xmlrpc_helpers.h new file:   champ/champ/package.xml new file:   champ/champ_base/.gitignore new file:   champ/champ_base/CMakeLists.txt new file:   champ/champ_base/config/ekf/base_to_footprint.yaml new file:   champ/champ_base/config/ekf/footprint_to_odom.yaml new file:   champ/champ_base/config/velocity_smoother/velocity_smoother.yaml new file:   champ/champ_base/include/actuator.h new file:   champ/champ_base/include/message_relay.h new file:   champ/champ_base/include/quadruped_controller.h new file:   champ/champ_base/include/state_estimation.h new file:   champ/champ_base/package.xml new file:   champ/champ_base/src/message_relay.cpp new file:   champ/champ_base/src/message_relay_node.cpp new file:   champ/champ_base/src/quadruped_controller.cpp new file:   champ/champ_base/src/quadruped_controller_node.cpp new file:   champ/champ_base/src/state_estimation.cpp new file:   champ/champ_base/src/state_estimation_node.cpp new file:   champ/champ_bringup/CMakeLists.txt new file:   champ/champ_bringup/champ_bringup/__init__.py new file:   champ/champ_bringup/champ_bringup/joint_calibrator_relay.py new file:   champ/champ_bringup/launch/bringup.launch new file:   champ/champ_bringup/launch/bringup.launch.py new file:   champ/champ_bringup/launch/include/laser/d435.launch new file:   champ/champ_bringup/launch/include/laser/hokuyo.launch new file:   champ/champ_bringup/launch/include/laser/kinect.launch new file:   champ/champ_bringup/launch/include/laser/lms1xx.launch new file:   champ/champ_bringup/launch/include/laser/realsense.launch new file:   champ/champ_bringup/launch/include/laser/rplidar.launch new file:   champ/champ_bringup/launch/include/laser/sim.launch new file:   champ/champ_bringup/launch/include/laser/sweep.launch new file:   champ/champ_bringup/launch/include/laser/xv11.launch new file:   champ/champ_bringup/launch/include/laser/ydlidar.launch new file:   champ/champ_bringup/launch/include/velocity_smoother.launch new file:   champ/champ_bringup/launch/joints_gui.launch new file:   champ/champ_bringup/launch/joints_gui.launch.py new file:   champ/champ_bringup/launch/openmutt_bringup.launch.py new file:   champ/champ_bringup/package.xml new file:   champ/champ_config/CMakeLists.txt new file:   champ/champ_config/config/autonomy/navigation.yaml new file:   champ/champ_config/config/autonomy/slam.yaml new file:   champ/champ_config/config/gait/gait.yaml new file:   champ/champ_config/config/joints/joints.yaml new file:   champ/champ_config/config/links/links.yaml new file:   champ/champ_config/include/gait_config.h new file:   champ/champ_config/include/hardware_config.h new file:   champ/champ_config/include/quadruped_description.h new file:   champ/champ_config/launch/bringup.launch.py new file:   champ/champ_config/launch/gazebo.launch.py new file:   champ/champ_config/launch/navigate.launch.py new file:   champ/champ_config/launch/slam.launch.py new file:   champ/champ_config/maps/map.pgm new file:   champ/champ_config/maps/map.yaml new file:   champ/champ_config/maps/playground.pgm new file:   champ/champ_config/maps/playground.yaml new file:   champ/champ_config/package.xml new file:   champ/champ_config/setup.bash new file:   champ/champ_config/worlds/default.world new file:   champ/champ_config/worlds/outdoor.world new file:   champ/champ_config/worlds/playground.world new file:   champ/champ_description/CMakeLists.txt new file:   champ/champ_description/environment/gz_sim_resource_path.dsv new file:   champ/champ_description/launch/description.launch new file:   champ/champ_description/launch/description.launch.py new file:   champ/champ_description/launch/view_urdf.launch new file:   champ/champ_description/meshes/arm/base.stl new file:   champ/champ_description/meshes/arm/lower_arm.stl new file:   champ/champ_description/meshes/arm/upper_arm.stl new file:   champ/champ_description/meshes/arm/wrist1.stl new file:   champ/champ_description/meshes/arm/wrist2.stl new file:   champ/champ_description/meshes/asus_camera_simple.dae new file:   champ/champ_description/meshes/base.stl new file:   champ/champ_description/meshes/base_simple.stl new file:   champ/champ_description/meshes/hip.stl new file:   champ/champ_description/meshes/hokuyo_utm_30lx.dae new file:   champ/champ_description/meshes/lower_leg.stl new file:   champ/champ_description/meshes/lower_leg_simple.stl new file:   champ/champ_description/meshes/upper_leg.stl new file:   champ/champ_description/meshes/upper_leg_simple.stl new file:   champ/champ_description/package.xml new file:   champ/champ_description/rviz/urdf_viewer.rviz new file:   champ/champ_description/urdf/accessories.urdf.xacro new file:   champ/champ_description/urdf/asus_camera.urdf.xacro new file:   champ/champ_description/urdf/champ.urdf new file:   champ/champ_description/urdf/champ.urdf.xacro new file:   champ/champ_description/urdf/champ_arm.urdf new file:   champ/champ_description/urdf/champ_velodyne.urdf new file:   champ/champ_description/urdf/gen_urdf new file:   champ/champ_description/urdf/hokuyo_utm30lx.urdf.xacro new file:   champ/champ_description/urdf/leg.urdf.xacro new file:   champ/champ_description/urdf/properties.urdf.xacro new file:   champ/champ_gazebo/CMakeLists.txt new file:   champ/champ_gazebo/config/gazebo.yaml new file:   champ/champ_gazebo/config/ros_control.yaml new file:   champ/champ_gazebo/launch/gazebo.launch.py new file:   champ/champ_gazebo/launch/spawn_robot.launch new file:   champ/champ_gazebo/launch/spawn_world.launch new file:   champ/champ_gazebo/package.xml new file:   champ/champ_gazebo/scripts/imu_sensor.py new file:   champ/champ_gazebo/scripts/odometry.py new file:   champ/champ_gazebo/scripts/odometry_tf.py new file:   champ/champ_gazebo/src/contact_sensor.cpp new file:   champ/champ_gazebo/worlds/default.world new file:   champ/champ_gazebo/worlds/outdoor.world new file:   champ/champ_gazebo/worlds/playground.world new file:   champ/champ_msgs/CMakeLists.txt new file:   champ/champ_msgs/msg/Contacts.msg new file:   champ/champ_msgs/msg/ContactsStamped.msg new file:   champ/champ_msgs/msg/Imu.msg new file:   champ/champ_msgs/msg/Joints.msg new file:   champ/champ_msgs/msg/PID.msg new file:   champ/champ_msgs/msg/Point.msg new file:   champ/champ_msgs/msg/PointArray.msg new file:   champ/champ_msgs/msg/Pose.msg new file:   champ/champ_msgs/msg/Velocities.msg new file:   champ/champ_msgs/package.xml new file:   champ/champ_navigation/CMakeLists.txt new file:   champ/champ_navigation/launch/navigate.launch.py new file:   champ/champ_navigation/launch/slam.launch.py new file:   champ/champ_navigation/package.xml new file:   champ/champ_navigation/rviz/navigation.rviz new file:   champ/champ_navigation/rviz/navigation_minimal.rviz new file:   champ/champ_navigation/rviz/slam.rviz new file:   champ/docs/images/leg_stretched.png new file:   champ/docs/images/navigation.gif new file:   champ/docs/images/robots.gif new file:   champ/docs/images/slam.gif new file:   champ_teleop/CMakeLists.txt new file:   champ_teleop/README.md new file:   champ_teleop/champ_teleop.py new file:   champ_teleop/launch/teleop.launch.py new file:   champ_teleop/package.xml new file:   manage_champ.sh new file:   openmutt_config/CMakeLists.txt new file:   openmutt_config/README.md new file:   openmutt_config/config.json new file:   openmutt_config/config/gait/gait.yaml new file:   openmutt_config/config/joints/joints.yaml new file:   openmutt_config/config/links/links.yaml new file:   openmutt_config/config/move_base/base_local_planner_holonomic_params.yaml new file:   openmutt_config/config/move_base/costmap_common_params.yaml new file:   openmutt_config/config/move_base/global_costmap_params.yaml new file:   openmutt_config/config/move_base/local_costmap_params.yaml new file:   openmutt_config/config/move_base/move_base_params.yaml new file:   openmutt_config/config/ros_control/ros_control.yaml new file:   openmutt_config/imuListener.py new file:   openmutt_config/include/gait_config.h new file:   openmutt_config/include/hardware_config.h new file:   openmutt_config/include/quadruped_description.h new file:   openmutt_config/jointTrajListener.py new file:   openmutt_config/launch/bringup.launch new file:   openmutt_config/launch/bringup.launch.py new file:   openmutt_config/launch/gazebo.launch new file:   openmutt_config/launch/include/amcl.launch new file:   openmutt_config/launch/include/gmapping.launch new file:   openmutt_config/launch/include/move_base.launch new file:   openmutt_config/launch/navigate.launch new file:   openmutt_config/launch/slam.launch new file:   openmutt_config/launch/spawn_robot.launch new file:   openmutt_config/legRQTPlotter.py new file:   openmutt_config/maps/map.pgm new file:   openmutt_config/maps/map.yaml new file:   openmutt_config/package.xml new file:   openmutt_config/setup.bash new file:   openmutt_config/worlds/default.world new file:   openmutt_config/worlds/outdoor.world new file:   openmutt_description/CMakeLists.txt new file:   openmutt_description/launch/description.launch.py new file:   openmutt_description/meshes/25-2525-751_6-CL-1.stl new file:   openmutt_description/meshes/25-2525-751_6-CL.stl new file:   openmutt_description/meshes/Body_Bearing-1.stl new file:   openmutt_description/meshes/Body_Bearing-2.stl new file:   openmutt_description/meshes/Body_Bearing-3.stl new file:   openmutt_description/meshes/Body_Bearing-4.stl new file:   openmutt_description/meshes/Body_Electrical-Leg-Tray-1.stl new file:   openmutt_description/meshes/Body_Electrical-Leg-Tray-2.stl new file:   openmutt_description/meshes/Body_Leg-Center-1.stl new file:   openmutt_description/meshes/Body_Leg-Center-2.stl new file:   openmutt_description/meshes/Body_Mid-BatteryCover-1.stl new file:   openmutt_description/meshes/Body_Mid-BatteryCover-2.stl new file:   openmutt_description/meshes/Body_Mid-EletricalPlate-1.stl new file:   openmutt_description/meshes/Body_Mid-TopCover-Side-1.stl new file:   openmutt_description/meshes/Body_Mid-TopCover-Side-2.stl new file:   openmutt_description/meshes/Cycloidal_Simplified_for_FEA-v1-1.stl new file:   openmutt_description/meshes/Cycloidal_Simplified_for_FEA-v1-2.stl new file:   openmutt_description/meshes/Cycloidal_Simplified_for_FEA-v1-3.stl new file:   openmutt_description/meshes/Cycloidal_Simplified_for_FEA-v1-4-1.stl new file:   openmutt_description/meshes/Cycloidal_Simplified_for_FEA-v1-4-2.stl new file:   openmutt_description/meshes/Cycloidal_Simplified_for_FEA-v1-4-3.stl new file:   openmutt_description/meshes/Cycloidal_Simplified_for_FEA-v1-4-4-1.stl new file:   openmutt_description/meshes/Cycloidal_Simplified_for_FEA-v1-4-4-2.stl new file:   openmutt_description/meshes/Cycloidal_Simplified_for_FEA-v1-4-4-3.stl new file:   openmutt_description/meshes/Cycloidal_Simplified_for_FEA-v1-4-4.stl new file:   openmutt_description/meshes/Cycloidal_Simplified_for_FEA-v1-4.stl new file:   openmutt_description/meshes/Cycloidal_Simplified_for_FEA-v1.stl new file:   openmutt_description/meshes/Hip_Main-Short-1-2.stl new file:   openmutt_description/meshes/Hip_Main-Short-1.stl new file:   openmutt_description/meshes/Hip_Main-Short-2-1.stl new file:   openmutt_description/meshes/Hip_Main-Short-2.stl new file:   openmutt_description/meshes/Leg_Knee-Cable-Top-Plate-V3.2-1.stl new file:   openmutt_description/meshes/Leg_Knee-Cable-Top-Plate-V3.2-2-1-1.stl new file:   openmutt_description/meshes/Leg_Knee-Cable-Top-Plate-V3.2-2-1.stl new file:   openmutt_description/meshes/Leg_Knee-Cable-Top-Plate-V3.2-2.stl new file:   openmutt_description/meshes/Leg_Knee-Cable-Top-V3.2-1-1.stl new file:   openmutt_description/meshes/Leg_Knee-Cable-Top-V3.2-1-2.stl new file:   openmutt_description/meshes/Leg_Knee-Cable-Top-V3.2-2-1.stl new file:   openmutt_description/meshes/Leg_Knee-Cable-Top-V3.2-2.stl new file:   openmutt_description/meshes/Leg_Knee-Cable-V3.2-1-1.stl new file:   openmutt_description/meshes/Leg_Knee-Cable-V3.2-1-2.stl new file:   openmutt_description/meshes/Leg_Knee-Cable-V3.2-2-1.stl new file:   openmutt_description/meshes/Leg_Knee-Cable-V3.2-2.stl new file:   openmutt_description/meshes/Leg_Knee-Cartilage-Outer-1-1.stl new file:   openmutt_description/meshes/Leg_Knee-Cartilage-Outer-1-2.stl new file:   openmutt_description/meshes/Leg_Knee-Cartilage-Outer-1-3.stl new file:   openmutt_description/meshes/Leg_Knee-Cartilage-Outer-2.stl new file:   openmutt_description/meshes/Leg_Shank-Bushing-1.stl new file:   openmutt_description/meshes/Leg_Shank-Bushing-2-1-1.stl new file:   openmutt_description/meshes/Leg_Shank-Bushing-2-1.stl new file:   openmutt_description/meshes/Leg_Shank-Bushing-2.stl new file:   openmutt_description/meshes/Leg_Thigh-1-1.stl new file:   openmutt_description/meshes/Leg_Thigh-1-2.stl new file:   openmutt_description/meshes/Leg_Thigh-2-1.stl new file:   openmutt_description/meshes/Leg_Thigh-2.stl new file:   openmutt_description/meshes/Leg_Thigh-Plate-1-1.stl new file:   openmutt_description/meshes/Leg_Thigh-Plate-1-2.stl new file:   openmutt_description/meshes/Leg_Thigh-Plate-2-1.stl new file:   openmutt_description/meshes/Leg_Thigh-Plate-2.stl new file:   openmutt_description/meshes/Master_TubeSuport-1.stl new file:   openmutt_description/meshes/Master_TubeSuport.stl new file:   openmutt_description/meshes/SD_Body_Leg-Bearing-1.stl new file:   openmutt_description/meshes/SD_Body_Leg-Bearing-2.stl new file:   openmutt_description/meshes/SD_Body_Leg-Motor-1.stl new file:   openmutt_description/meshes/SD_Body_Leg-Motor-2.stl new file:   openmutt_description/meshes/SD_Body_Mid-Brace-1.stl new file:   openmutt_description/meshes/SD_Body_Mid-Brace-2.stl new file:   openmutt_description/meshes/SD_Body_Mid-ELECTRICAL-BulkHead-1.stl new file:   openmutt_description/meshes/SD_Body_Mid-ELECTRICAL-BulkHead-2.stl new file:   openmutt_description/meshes/SD_Body_Mid-TopPlate-Center-1.stl new file:   openmutt_description/meshes/SD_Hip_motor_mount-1-1.stl new file:   openmutt_description/meshes/SD_Hip_motor_mount-1-2.stl new file:   openmutt_description/meshes/SD_Hip_motor_mount-2-1.stl new file:   openmutt_description/meshes/SD_Hip_motor_mount-2.stl new file:   openmutt_description/meshes/SD_TPU_Foot-1-2.stl new file:   openmutt_description/meshes/SD_TPU_Foot-1.stl new file:   openmutt_description/meshes/SD_TPU_Foot-2-1.stl new file:   openmutt_description/meshes/SD_TPU_Foot-2.stl new file:   openmutt_description/meshes/SD_foot-1-1-2.stl new file:   openmutt_description/meshes/SD_foot-1-1.stl new file:   openmutt_description/meshes/SD_foot-1-2-1.stl new file:   openmutt_description/meshes/SD_foot-1-2.stl new file:   openmutt_description/meshes/SD_ideler-1-2.stl new file:   openmutt_description/meshes/SD_ideler-1.stl new file:   openmutt_description/meshes/SD_ideler-2-1.stl new file:   openmutt_description/meshes/SD_ideler-2.stl new file:   openmutt_description/meshes/SD_shank-main-V2-1-1.stl new file:   openmutt_description/meshes/SD_shank-main-V2-1-2.stl new file:   openmutt_description/meshes/SD_shank-main-V2-2-1.stl new file:   openmutt_description/meshes/SD_shank-main-V2-2.stl new file:   openmutt_description/meshes/Sd_Body_Mid-Sideplate-1.stl new file:   openmutt_description/meshes/Sd_Body_Mid-Sideplate-2.stl new file:   openmutt_description/meshes/base_link.stl new file:   openmutt_description/package.xml new file:   openmutt_description/rviz/urdf.rviz new file:   openmutt_description/urdf/MASTER.urdf new file:   openmutt_description/urdf/openMuttSensors.urdf

File: openmutt_description/urdf/openMuttSensors.urdf (robot description, URDF)
Before this commit: robot openMutt, 46 links, 45 joints
Links:
- link backLeftFoot: geometry collision sphere radius=0.032; visual sphere radius=0.032
- link backRightFoot: geometry collision sphere radius=0.032; visual sphere radius=0.032
- link frontLeftFoot: geometry collision sphere radius=0.032; visual sphere radius=0.032
- link frontRightFoot: geometry collision sphere radius=0.032; visual sphere radius=0.032
